Commit message: backup 2704

File: catkin_ws/src/antenna/antenna_description/urdf/antenna.xacro (robot description, xacro)
@@ -27,7 +27,7 @@
       <mass value="${mass}"/>
       <inertia
-	  ixx="1" ixy="0.0" ixz="0.0"
-	  iyy="1" iyz="0.0"
-	  izz="1"/>
+  	  ixx="1" ixy="0.0" ixz="0.0"
+  	  iyy="1" iyz="0.0"
+  	  izz="1"/>
     </inertial>
   </link>
@@ -45,5 +45,5 @@
       <origin xyz="0 0 0" rpy="0 0 0"/>
       <geometry>
-	<box size="0.1 0.1 0.8"/>
+        <box size="0.1 0.1 0.8"/>
       </geometry>
     </collision>
@@ -51,5 +51,5 @@
       <origin xyz="0 0 0" rpy="0 0 0"/>
       <geometry>
-	<box size="0.1 0.1 0.8"/>
+        <box size="0.1 0.1 0.8"/>
       </geometry>
     </visual>
@@ -58,7 +58,7 @@
       <mass value="${mass * 4.69}"/>
       <inertia
-	  ixx="0.25" ixy="0.0" ixz="0.0"
-	  iyy="0.25" iyz="0.0"
-	  izz="0.006"/>
+  	  ixx="0.25" ixy="0.0" ixz="0.0"
+  	  iyy="0.25" iyz="0.0"
+  	  izz="0.006"/>
     </inertial>
   </link>
@@ -69,5 +69,5 @@
     <origin xyz="0 0 0.45" rpy="0 ${pi / (-2)} 0"/>
     <axis xyz="0 1 0"/>
-    <limit effort="30" lower="0" upper="${pi}" velocity="0.02094"/>
+    <limit effort="30" lower="0" upper="${pi}" velocity="0"/>
     <dynamics damping="0" friction="10"/>
   </joint>
@@ -77,5 +77,5 @@
       <origin xyz="0 0 0" rpy="0 0 0"/>
       <geometry>
-	<box size="0.1 0.8 0.2"/>
+      	<box size="0.1 0.8 0.2"/>
       </geometry>
     </collision>
@@ -83,5 +83,5 @@
       <origin xyz="0 0 0" rpy="0 0 0"/>
       <geometry>
-	<box size="0.1 0.8 0.2"/>
+      	<box size="0.1 0.8 0.2"/>
       </geometry>
     </visual>
@@ -90,7 +90,7 @@
       <mass value="${mass * pi / 2}"/>
       <inertia
-	  ixx="0.0884" ixy="0.0" ixz="0.0"
-	  iyy="0.0065" iyz="0.0"
-	  izz="0.0845"/>
+  	  ixx="0.0884" ixy="0.0" ixz="0.0"
+  	  iyy="0.0065" iyz="0.0"
+  	  izz="0.0845"/>
     </inertial>
   </link>

Commit message: backup 1oo5

File: catkin_ws/src/antenna/antenna_description/urdf/antenna.xacro (robot description, xacro)
@@ -69,5 +69,5 @@
     <origin xyz="0 0 0.45" rpy="0 ${pi / (-2)} 0"/>
     <axis xyz="0 1 0"/>
-    <limit effort="30" lower="0" upper="${pi}" velocity="0"/>
+    <limit effort="30" lower="0" upper="${pi}" velocity="10"/>
     <dynamics damping="0" friction="10"/>
   </joint>
